File: Blinker Baseboard RP2040/Blinker Baseboard RP2040.kicad_pcb (KiCad board)
At the start: 2 copper layers, 52 x 60 mm, 74 parts, among them J1 USB_B_Micro, J2 Conn_01x02, J3 Charger - Out, J4 Charger - In, J5 Charger - Bat, J6 L Spinner, J7 R Spinner, J8 L Blinker, J9 R Blinker, Q1 BSS138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

Commit message: r1
Other:
- board text added: "Blinker, Baseboard RP2040 v1.0 r1 Jim 2024-02-17"
