File: Blinker Spinner/Blinker.kicad_pcb (KiCad board)
At the start: 2 copper layers, 35 x 35 mm, 17 parts, among them J1 To Base

Commit message: r1
Other:
- board text added: "Blinker, round v1.0 r1"
- board text added: "Jim, 2024-02-17"
- board text removed: "Blinker, round v1.0"
- board text removed: "Jim, 2024-02-03"
Changed lines of the file:
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@@
   (gr_circle (center 100 100) (end 110 100)
     (stroke (width 0.1) (type default)) (fill none) (layer "Edge.Cuts"))
-  (gr_text "Blinker, round v1.0" (at 110.5 93 270) (layer "F.SilkS")
+  (gr_text "Blinker, round v1.0 r1" (at 110.5 91.5 270) (layer "F.SilkS")
     (effects (font (size 1 1) (thickness 0.15)) (justify left bottom))
   )
-  (gr_text "Jim, 2024-02-03" (at 89.5 107.5 90) (layer "F.SilkS")
+  (gr_text "Jim, 2024-02-17" (at 89.5 107.5 90) (layer "F.SilkS")
     (effects (font (size 1 1) (thickness 0.15)) (justify left bottom))
   )
