File: Blinker Baseboard/Blinker Baseboard.kicad_sch (KiCad schematic)
At the start: 47 parts, among them J1 L Spinner, J2 R Spinner, J3 L Blinker, J4 R Blinker, J5 Charger - Out, J6 Charger - In, J7 Charger - Bat, Q1 BSS138, Q10 BSS138, Q11 BSS138, Q12 BSS138, Q2 BSS138, Q3 BSS138, Q4 BSS138, Q5 BSS138, Q6 BSS138, Q7 BSS138, Q8 BSS138, Q9 BSS138, SW1 SW_Push, U1 RaspberryPi_Pico

Commit message: Baseboard rework
R2 became v2.
Parts:
- removed J5: Charger - Out, Connector_PinHeader_2.54mm:PinHeader_1x02_P2.54mm_Vertical, symbol Connector_Generic:Conn_01x02
- removed J6: Charger - In, Connector_PinHeader_2.54mm:PinHeader_1x02_P2.54mm_Vertical, symbol Connector_Generic:Conn_01x02
- removed J7: Charger - Bat, Connector_PinHeader_2.54mm:PinHeader_1x03_P2.54mm_Vertical, symbol Connector_Generic:Conn_01x03
- added C1, C10, C2, C3, C4, C5, C6, C7, C8, C9: C, Capacitor_SMD:C_0805_2012Metric_Pad1.18x1.45mm_HandSolder, symbol Device:C
- added D1, D2: LED, LED_SMD:LED_0805_2012Metric_Pad1.15x1.40mm_HandSolder, symbol Device:LED
- added R27, R28: R, Resistor_SMD:R_0805_2012Metric_Pad1.20x1.40mm_HandSolder, symbol Device:R
- added U2: ~, ek:Electrokit LiPo charger, symbol Battery_Management:Electrokit_LiPo_Charger
- J1, J2: footprint Connector_Molex:Molex_PicoBlade_53047-0510_1x05_P1.25mm_Vertical -> Connector_PinHeader_2.54mm:PinHeader_1x05_P2.54mm_Vertical
- J3, J4: footprint Connector_Molex:Molex_PicoBlade_53047-0310_1x03_P1.25mm_Vertical -> Connector_PinHeader_2.54mm:PinHeader_1x03_P2.54mm_Vertical
- R1, R10, R11, R12, R13, R14, R15, R16, R17, R18, R19, R2, R20, R21, R22, R23, R24, R25, R26, R3, R4, R5, R6, R7, R8, R9: footprint Resistor_SMD:R_1206_3216Metric -> Resistor_SMD:R_0805_2012Metric_Pad1.20x1.40mm_HandSolder
Connections:
- net GND: now also C1.2, C10.2, C2.2, C3.2, C4.2, C5.2, C6.2, C7.2, C8.2, C9.2, D1.1 (K), R28.1, U2.4 (Out_-)
- net VCC: now also C1.1, C10.1, C2.1, C3.1, C4.1, C5.1, C6.1, C7.1, C8.1, C9.1, R27.2
- net at U1.29 (GPIO22): now also D2.2 (A)
- net at SW1.2: now also U2.3 (Out_+)
- new net: D2.1 (K), R28.2
- new net: D1.2 (A), R27.1
- no-connect marks 0 -> 22
Other:
- moved on the sheet: U1
